File: pcb/ESP3232_to_GW1NS2C/source/brekout_board.brd (EAGLE design)
At the start: 53.2 x 32.5 mm, 3 parts

Commit message: 2 layer PCB update
Routing:
- net RX2: track 57.9 -> 66.9 mm
- net D35: track 40.3 -> 38.0 mm
- added copper zone on layer 1, net GND
- added copper zone on layer 16, net GND
- removed copper zone on layer 2, net GND
- removed copper zone on layer 15, net PWR
Other:
- board text added: "1"
- board text added: "15"
- board text added: "19"
- board text added: "2"
- board text added: "20"
Changed lines of the file:
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@@
 <wire x1="53.23" y1="32.49" x2="0" y2="32.49" width="0" layer="20"/>
 <wire x1="0" y1="32.49" x2="0" y2="0" width="0" layer="20"/>
+<text x="4.5" y="25" size="1.778" layer="21">1</text>
+<text x="4.5" y="6" size="1.778" layer="21">1</text>
+<text x="39.5" y="25" size="1.778" layer="21">15</text>
+<text x="39.5" y="6" size="1.778" layer="21">15</text>
+<text x="51" y="27" size="1.778" layer="21">2</text>
+<text x="50" y="1.5" size="1.778" layer="21">20</text>
+<text x="44" y="1.5" size="1.778" layer="21">19</text>
+<text x="44.5" y="27" size="1.778" layer="21">1</text>
 </plain>
 <attributes>
@@
 necessary adjustments and save your customized
 design rules under a new name.</description>
-<param name="layerSetup" value="(1*2*15*16)"/>
+<param name="layerSetup" value="(1*16)"/>
 <param name="mtCopper" value="0.035mm 0.035mm 0.035mm 0.035mm 0.035mm 0.035mm 0.035mm 0.035mm 0.035mm 0.035mm 0.035mm 0.035mm 0.035mm 0.035mm 0.035mm 0.035mm"/>
 <param name="mtIsolate" value="1.5mm 0.15mm 0.2mm 0.15mm 0.2mm 0.15mm 0.2mm 0.15mm 0.2mm 0.15mm 0.2mm 0.15mm 0.2mm 0.15mm 0.2mm"/>
@@
 <elements>
 <element name="J1" library="pinhead" library_urn="urn:adsk.eagle:library:325" package="2X10" package3d_urn="urn:adsk.eagle:package:22405/2" value="" x="48.31" y="16.17" rot="R270">
-<attribute name="NAME" x="49.63" y="29.485" size="1.27" layer="25" ratio="10"/>
+<attribute name="NAME" x="47.63" y="29.485" size="1.27" layer="25" ratio="10"/>
 <attribute name="VALUE" x="43.865" y="28.87" size="1.27" layer="27" rot="R270"/>
 </element>
@@
 <contactref element="J3" pad="6"/>
 <contactref element="J1" pad="4"/>
-<wire x1="20.0025" y1="1.5875" x2="17.78" y2="3.81" width="0.3048" layer="1"/>
-<wire x1="50.8" y1="1.5875" x2="20.0025" y2="1.5875" width="0.3048" layer="1"/>
-<wire x1="50.8" y1="23.8125" x2="50.8" y2="1.5875" width="0.3048" layer="1"/>
-<wire x1="49.8475" y1="24.765" x2="50.8" y2="23.8125" width="0.3048" layer="1"/>
-<wire x1="49.8475" y1="24.765" x2="49.58" y2="25.06" width="0.3048" layer="1"/>
+<wire x1="17.78" y1="3.81" x2="27.47" y2="13.5" width="0.3048" layer="1"/>
+<wire x1="27.47" y1="13.5" x2="39" y2="13.5" width="0.3048" layer="1"/>
+<wire x1="50.7992" y1="7.7850125" x2="50.0850125" y2="8.4992" width="0.3048" layer="1"/>
+<wire x1="39" y1="13.5" x2="41.1679" y2="11.3321" width="0.3048" layer="1"/>
+<wire x1="41.1679" y1="11.3321" x2="41.1679" y2="8.02578125" width="0.3048" layer="1"/>
+<wire x1="41.1679" y1="8.02578125" x2="46.31078125" y2="2.8829" width="0.3048" layer="1"/>
+<wire x1="46.31078125" y1="2.8829" x2="49.4471125" y2="2.8829" width="0.3048" layer="1"/>
+<wire x1="49.4471125" y1="2.8829" x2="50.7992" y2="4.2349875" width="0.3048" layer="1"/>
+<wire x1="50.7992" y1="4.2349875" x2="50.7992" y2="7.7850125" width="0.3048" layer="1"/>
+<wire x1="50.0850125" y1="8.4992" x2="49.0749875" y2="8.4992" width="0.3048" layer="1"/>
+<wire x1="49.0749875" y1="8.4992" x2="48.3608" y2="9.2133875" width="0.3048" layer="1"/>
+<wire x1="48.3608" y1="23.8408" x2="49.58" y2="25.06" width="0.3048" layer="1"/>
+<wire x1="48.3608" y1="9.2133875" x2="48.3608" y2="23.8408" width="0.3048" layer="1"/>
 </signal>
 <signal name="TX2">
@@
 <wire x1="49.53" y1="27.6225" x2="49.58" y2="27.6" width="0.3048" layer="16"/>
 <wire x1="7.62" y1="28.8925" x2="7.62" y2="28.81" width="0.3048" layer="16"/>
-<polygon width="0.1524" layer="2">
+<polygon width="0.1524" layer="16">
 <vertex x="0.5" y="0.5"/>
 <vertex x="52.5" y="0.5"/>
@@
 <vertex x="1.5" y="31.5"/>
 <vertex x="0.5" y="30.5"/>
+</polygon>
+<polygon width="0.1524" layer="1">
+<vertex x="0.5" y="1"/>
+<vertex x="52.5" y="1"/>
+<vertex x="52.5" y="31"/>
+<vertex x="51.5" y="32"/>
+<vertex x="1.5" y="32"/>
+<vertex x="0.5" y="31"/>
 </polygon>
 </signal>
@@
 <wire x1="48.26" y1="6.0325" x2="47.3075" y2="6.985" width="0.3048" layer="1"/>
 <wire x1="48.26" y1="4.1275" x2="48.26" y2="6.0325" width="0.3048" layer="1"/>
-<wire x1="47.625" y1="3.4925" x2="48.26" y2="4.1275" width="0.3048" layer="1"/>
-<wire x1="41.91" y1="3.4925" x2="47.625" y2="3.4925" width="0.3048" layer="1"/>
-<wire x1="41.91" y1="17.145" x2="41.91" y2="3.4925" width="0.3048" layer="1"/>
-<wire x1="30.48" y1="28.575" x2="41.91" y2="17.145" width="0.3048" layer="1"/>
+<wire x1="47.625" y1="3.4925" x2="47.81625" y2="3.68375" width="0.3048" layer="1"/>
+<wire x1="47.81625" y1="3.68375" x2="48.26" y2="4.1275" width="0.3048" layer="1"/>
+<wire x1="30.48" y1="28.575" x2="41.7775" y2="17.2775" width="0.3048" layer="1"/>
+<wire x1="41.7775" y1="17.2775" x2="41.91" y2="17.145" width="0.3048" layer="1"/>
 <wire x1="47.3075" y1="6.985" x2="47.04" y2="7.28" width="0.3048" layer="1"/>
 <wire x1="30.48" y1="28.575" x2="30.48" y2="28.81" width="0.3048" layer="1"/>
+<wire x1="46.5349875" y1="3.5208" x2="47.5450125" y2="3.5208" width="0.3048" layer="1"/>
+<wire x1="47.5450125" y1="3.5208" x2="47.7079625" y2="3.68375" width="0.3048" layer="1"/>
+<wire x1="47.7079625" y1="3.68375" x2="47.81625" y2="3.68375" width="0.3048" layer="1"/>
+<wire x1="41.7775" y1="8.2782875" x2="46.5349875" y2="3.5208" width="0.3048" layer="1"/>
+<wire x1="41.7775" y1="17.2775" x2="41.7775" y2="8.2782875" width="0.3048" layer="1"/>
 </signal>
 <signal name="D34">
@@
 <contactref element="J2" pad="15"/>
 </signal>
-<signal name="PWR">
-<polygon width="0.1524" layer="15">
-<vertex x="0.5" y="1"/>
-<vertex x="52.5" y="1"/>
-<vertex x="52.5" y="31"/>
-<vertex x="51.5" y="32"/>
-<vertex x="1.5" y="32"/>
-<vertex x="0.5" y="31"/>
-</polygon>
-</signal>
 </signals>
